File: hardware/ATTinyBreakout.sch (EAGLE design)
At the start: 15 parts, among them U1 TINY85-20-DIP

Commit message: Revision with 3 pin headers (Ludus style)
Parts:
- added JP5, JP6: (no value), SparkFun-Connectors:M04LOCK
- added STANDOFF3, STANDOFF4: STAND-OFF, SparkFun-Electromechanical:STAND-OFF
- added U$2: SFE_LUDUSSFE_LUDUS-M, SparkFun-Aesthetics:SFE_LUDUSSFE_LUDUS-M
- D1: device SparkFun-LED:LED-BLUE0603 -> SparkFun-LED:LED-BLUE1206
Connections:
- removed net SWITCHED_VCC: JP2.1, S1.2, S1.5, U1.VCC
- new net N$3: JP2.4, JP5.1, JP5.2, JP5.3, JP5.4, JP6.1, JP6.2, JP6.3, JP6.4, S1.2, S1.5, U1.VCC
- net PB0_MOSI: now also JP2.1; no longer JP2.4
- net PB1_MISO: now also JP2.2; no longer JP2.3
- net PB2_SCK: now also JP2.3; no longer JP2.2
Other:
- moved on the sheet: JP2
